File: PCB/full-keyboard.kicad_sch (KiCad schematic)
At the start: 0 parts

Commit message: Started laying out the schematic and found the library for the switches i am going to use.
Parts:
- added A1: RaspberryPi_Pico, Module:RaspberryPi_Pico_Common_Unspecified, symbol MCU_Module:RaspberryPi_Pico
- added U1: MCP23017-E_SP, Package_SO:SOIC-28W_7.5x17.9mm_P1.27mm, symbol MCP23017-E_SP:MCP23017-E_SP
Connections:
- new net 3V3(OUT): A1.36 (3V3), U1.18 (~{RESET})
- new net GND: A1.13 (GND), A1.18 (GND), A1.23 (GND), A1.28 (GND), A1.3 (GND), A1.38 (GND), A1.8 (GND), U1.15 (A0), U1.16 (A1), U1.17 (A2)
- new net SCL: A1.2 (GPIO1), U1.12 (SCK)
- new net SDA: A1.1 (GPIO0), U1.13 (SDA)
Other:
- title: (none) -> Custom Keyboard

Commit message: started work on the schematic. got all the switches layed out
Parts:
- added D1, D10, D100, D101, D102, D103, D104, D105, D106, D107, D108, D11, D12, D13, D14, D15, D16, D17, D18, D19, D2, D20, D21, D22, D23, D24, D25, D26, D27, D28, D29, D3, D30, D31, D32, D33, D34, D35, D36, D37, D38, D39, D4, D40, D41, D42, D43, D44, D45, D46, D47, D48, D49, D5, D50, D51, D52, D53, D54, D55, D56, D57, D58, D59, D6, D60, D61, D62, D63, D64, D65, D66, D67, D68, D69, D7, D70, D71, D72, D73, D74, D75, D76, D77, D78, D79, D8, D80, D81, D82, D83, D84, D85, D86, D87, D88, D89, D9, D90, D91, D92, D93, D94, D95, D96, D97, D98, D99: D, symbol Device:D
- added J1: Conn_01x04_Pin, KiCad-SSD1306-0.91-OLED-4pin-128x32:SSD1306-0.91-OLED-4pin-128x32, symbol Connector:Conn_01x04_Pin
- added SW1, SW10, SW100, SW101, SW102, SW103, SW104, SW105, SW106, SW107, SW108, SW11, SW12, SW13, SW14, SW15, SW16, SW17, SW18, SW19, SW2, SW20, SW21, SW22, SW23, SW24, SW25, SW26, SW27, SW28, SW29, SW3, SW30, SW31, SW32, SW33, SW34, SW35, SW36, SW37, SW38, SW39, SW4, SW40, SW41, SW42, SW43, SW44, SW45, SW46, SW47, SW48, SW49, SW5, SW50, SW51, SW52, SW53, SW54, SW55, SW56, SW57, SW58, SW59, SW6, SW60, SW61, SW62, SW63, SW64, SW65, SW66, SW67, SW68, SW69, SW7, SW70, SW71, SW72, SW73, SW74, SW75, SW76, SW77, SW78, SW79, SW8, SW80, SW81, SW82, SW83, SW84, SW85, SW86, SW87, SW88, SW89, SW9, SW90, SW91, SW92, SW93, SW94, SW95, SW96, SW97, SW98, SW99: SW_Push, key-switches:SW_MX_Kailh_Choc_V1V2_THT_Hybrid, symbol Switch:SW_Push
Connections:
- net COL5: now reaches A1.10 (GPIO7)
- net COL5: now also SW24.1, SW42.1, SW6.1, SW60.1, SW78.1, SW96.1
- net COL6: now reaches A1.11 (GPIO8)
- net COL6: now also SW25.1, SW43.1, SW61.1, SW7.1, SW79.1, SW97.1
- net COL7: now reaches A1.12 (GPIO9)
- net COL7: now also SW26.1, SW44.1, SW62.1, SW8.1, SW80.1, SW98.1
- net COL8: now reaches A1.14 (GPIO10)
- net COL8: now also SW27.1, SW45.1, SW63.1, SW81.1, SW9.1, SW99.1
- net COL9: now reaches A1.15 (GPIO11)
- net COL9: now also SW10.1, SW100.1, SW28.1, SW46.1, SW64.1, SW82.1
- net COL10: now reaches A1.16 (GPIO12)
- net COL10: now also SW101.1, SW11.1, SW29.1, SW47.1, SW65.1, SW83.1
- net COL11: now reaches A1.17 (GPIO13)
- net COL11: now also SW102.1, SW12.1, SW30.1, SW48.1, SW66.1, SW84.1
- net COL13: now reaches A1.19 (GPIO14)
- net COL13: now also SW104.1, SW14.1, SW32.1, SW50.1, SW68.1, SW86.1
- net COL14: now reaches A1.20 (GPIO15)
- net COL14: now also SW105.1, SW15.1, SW33.1, SW51.1, SW69.1, SW87.1
- net COL15: now reaches A1.21 (GPIO16)
- net COL15: now also SW106.1, SW16.1, SW34.1, SW52.1, SW70.1, SW88.1
- net COL16: now reaches A1.22 (GPIO17)
- net COL16: now also SW107.1, SW17.1, SW35.1, SW53.1, SW71.1, SW89.1
- net COL17: now reaches A1.24 (GPIO18)
- net COL17: now also SW108.1, SW18.1, SW36.1, SW54.1, SW72.1, SW90.1
- net ROW0: now reaches A1.25 (GPIO19)
- net ROW0: now also D1.1 (K), D10.1 (K), D11.1 (K), D12.1 (K), D13.1 (K), D14.1 (K), D15.1 (K), D16.1 (K), D17.1 (K), D18.1 (K), D2.1 (K), D3.1 (K), D4.1 (K), D5.1 (K), D6.1 (K), D7.1 (K), D8.1 (K), D9.1 (K)
- net ROW1: now reaches A1.26 (GPIO20)
- net ROW1: now also D19.1 (K), D20.1 (K), D21.1 (K), D22.1 (K), D23.1 (K), D24.1 (K), D25.1 (K), D26.1 (K), D27.1 (K), D28.1 (K), D29.1 (K), D30.1 (K), D31.1 (K), D32.1 (K), D33.1 (K), D34.1 (K), D35.1 (K), D36.1 (K)
- net ROW2: now reaches A1.27 (GPIO21)
- net ROW2: now also D37.1 (K), D38.1 (K), D39.1 (K), D40.1 (K), D41.1 (K), D42.1 (K), D43.1 (K), D44.1 (K), D45.1 (K), D46.1 (K), D47.1 (K), D48.1 (K), D49.1 (K), D50.1 (K), D51.1 (K), D52.1 (K), D53.1 (K), D54.1 (K)
- net ROW3: now reaches A1.29 (GPIO22)
- net ROW3: now also D55.1 (K), D56.1 (K), D57.1 (K), D58.1 (K), D59.1 (K), D60.1 (K), D61.1 (K), D62.1 (K), D63.1 (K), D64.1 (K), D65.1 (K), D66.1 (K), D67.1 (K), D68.1 (K), D69.1 (K), D70.1 (K), D71.1 (K), D72.1 (K)
- net ROW4: now reaches A1.31 (GPIO26_ADC0)
- net ROW4: now also D73.1 (K), D74.1 (K), D75.1 (K), D76.1 (K), D77.1 (K), D78.1 (K), D79.1 (K), D80.1 (K), D81.1 (K), D82.1 (K), D83.1 (K), D84.1 (K), D85.1 (K), D86.1 (K), D87.1 (K), D88.1 (K), D89.1 (K), D90.1 (K)
- net ROW5: now reaches A1.32 (GPIO27_ADC1)
- net ROW5: now also D100.1 (K), D101.1 (K), D102.1 (K), D103.1 (K), D104.1 (K), D105.1 (K), D106.1 (K), D107.1 (K), D108.1 (K), D91.1 (K), D92.1 (K), D93.1 (K), D94.1 (K), D95.1 (K), D96.1 (K), D97.1 (K), D98.1 (K), D99.1 (K)
- net COL0: now reaches A1.4 (GPIO2)
- net COL0: now also SW1.1, SW19.1, SW37.1, SW55.1, SW73.1, SW91.1
- net COL1: now reaches A1.5 (GPIO3)
- net COL1: now also SW2.1, SW20.1, SW38.1, SW56.1, SW74.1, SW92.1
- net COL2: now reaches A1.6 (GPIO4)
- net COL2: now also SW21.1, SW3.1, SW39.1, SW57.1, SW75.1, SW93.1
- net COL3: now reaches A1.7 (GPIO5)
- net COL3: now also SW22.1, SW4.1, SW40.1, SW58.1, SW76.1, SW94.1
- net COL4: now reaches A1.9 (GPIO6)
- net COL4: now also SW23.1, SW41.1, SW5.1, SW59.1, SW77.1, SW95.1
- new net: D66.2 (A), SW66.2
- new net: D10.2 (A), SW10.2
- new net: D76.2 (A), SW76.2
- new net: D83.2 (A), SW83.2
- new net: D59.2 (A), SW59.2
- new net: D36.2 (A), SW36.2
- new net: D82.2 (A), SW82.2
- new net: D60.2 (A), SW60.2
- new net: D89.2 (A), SW89.2
- new net: D34.2 (A), SW34.2
- new net: D61.2 (A), SW61.2
- new net: D71.2 (A), SW71.2
- new net: D68.2 (A), SW68.2
- new net: D90.2 (A), SW90.2
- new net: D98.2 (A), SW98.2
- new net: D31.2 (A), SW31.2
- new net: D84.2 (A), SW84.2
- new net: D51.2 (A), SW51.2
- new net: D104.2 (A), SW104.2
- new net: D42.2 (A), SW42.2
- new net: D4.2 (A), SW4.2
- new net: D25.2 (A), SW25.2
- new net: D49.2 (A), SW49.2
- new net: D13.2 (A), SW13.2
- new net: D46.2 (A), SW46.2
- new net: D14.2 (A), SW14.2
- new net: D77.2 (A), SW77.2
- new net: D11.2 (A), SW11.2
- new net: D108.2 (A), SW108.2
- new net: D44.2 (A), SW44.2
- new net: D7.2 (A), SW7.2
- new net: D70.2 (A), SW70.2
- new net: D79.2 (A), SW79.2
- new net: D21.2 (A), SW21.2
- new net: D28.2 (A), SW28.2
- new net: D6.2 (A), SW6.2
- new net: D3.2 (A), SW3.2
- new net: D101.2 (A), SW101.2
- new net: D62.2 (A), SW62.2
- new net: D93.2 (A), SW93.2
- new net: D39.2 (A), SW39.2
- new net: D47.2 (A), SW47.2
- new net: D105.2 (A), SW105.2
- new net: D78.2 (A), SW78.2
- new net: D53.2 (A), SW53.2
- new net: D92.2 (A), SW92.2
- new net: D69.2 (A), SW69.2
- new net: D35.2 (A), SW35.2
- new net: D41.2 (A), SW41.2
- new net: D75.2 (A), SW75.2
- new net: D24.2 (A), SW24.2
- new net: D58.2 (A), SW58.2
- new net: D19.2 (A), SW19.2
- new net: D38.2 (A), SW38.2
- new net: D95.2 (A), SW95.2
- new net: D52.2 (A), SW52.2
- new net: D100.2 (A), SW100.2
- new net: D29.2 (A), SW29.2
- new net: D65.2 (A), SW65.2
- new net: D94.2 (A), SW94.2
- new net: D103.2 (A), SW103.2
- new net: D97.2 (A), SW97.2
- new net: D16.2 (A), SW16.2
- new net: D33.2 (A), SW33.2
- new net: D45.2 (A), SW45.2
- new net: D88.2 (A), SW88.2
- new net: D2.2 (A), SW2.2
- new net: D17.2 (A), SW17.2
- new net: D107.2 (A), SW107.2
- new net: D12.2 (A), SW12.2
- new net: D18.2 (A), SW18.2
- new net: D91.2 (A), SW91.2
- new net: D22.2 (A), SW22.2
- new net: D64.2 (A), SW64.2
- new net: D56.2 (A), SW56.2
- new net: D20.2 (A), SW20.2
- new net: D86.2 (A), SW86.2
- new net: D26.2 (A), SW26.2
- new net: D40.2 (A), SW40.2
- new net: D5.2 (A), SW5.2
- new net: D102.2 (A), SW102.2
- new net: D48.2 (A), SW48.2
- new net: D85.2 (A), SW85.2
- new net: D54.2 (A), SW54.2
- new net: D99.2 (A), SW99.2
- new net: D74.2 (A), SW74.2
- new net: D87.2 (A), SW87.2
- new net: D23.2 (A), SW23.2
- new net: D8.2 (A), SW8.2
- new net: D73.2 (A), SW73.2
- new net: D30.2 (A), SW30.2
- new net: D96.2 (A), SW96.2
- new net: D50.2 (A), SW50.2
- new net: D80.2 (A), SW80.2
- new net: D27.2 (A), SW27.2
- new net: D63.2 (A), SW63.2
- new net: D1.2 (A), SW1.2
- new net: D43.2 (A), SW43.2
- new net: D32.2 (A), SW32.2
- new net: D81.2 (A), SW81.2
- new net: D57.2 (A), SW57.2
- new net: D55.2 (A), SW55.2
- new net: D72.2 (A), SW72.2
- new net: D15.2 (A), SW15.2
- new net: D67.2 (A), SW67.2
- new net: D37.2 (A), SW37.2
- new net: D9.2 (A), SW9.2
- new net: D106.2 (A), SW106.2
- new net COL12: SW103.1, SW13.1, SW31.1, SW49.1, SW67.1, SW85.1
Other:
- moved on the sheet: A1, U1

Commit message: added BOM and added the leds to the schematic
Parts:
- added D109, D110, D111, D112, D113, D114, D115, D116, D117, D118, D119, D120, D121, D122, D123, D124, D125, D126, D127, D128, D129, D130, D131, D132, D133, D134, D135, D136, D137, D138, D139, D140, D141, D142, D143, D144, D145, D146, D147, D148, D149, D150, D151, D152, D153, D154, D155, D156, D157, D158, D159, D160, D161, D162, D163, D164, D165, D166, D167, D168, D169, D170, D171, D172, D173, D174, D175, D176, D177, D178, D179, D180, D181, D182, D183, D184, D185, D186, D187, D188, D189, D190, D191, D192, D193, D194, D195, D196, D197, D198, D199, D200, D201, D202, D203, D204, D205, D206, D207, D208, D209, D210, D211, D212, D213, D214, D215, D216: SK6812, LED_SMD:LED_SK6812_PLCC4_5.0x5.0mm_P3.2mm, symbol LED:SK6812
Connections:
- net GND: now also J1.1 (Pin_1), U1.10 (VSS), D109.1 (VSS), D110.1 (VSS), D111.1 (VSS), D112.1 (VSS), D113.1 (VSS), D114.1 (VSS), D115.1 (VSS), D116.1 (VSS), D117.1 (VSS), D118.1 (VSS), D119.1 (VSS), D120.1 (VSS), D121.1 (VSS), D122.1 (VSS), D123.1 (VSS), D124.1 (VSS), D125.1 (VSS), D126.1 (VSS), D127.1 (VSS), D128.1 (VSS), D129.1 (VSS), D130.1 (VSS), D131.1 (VSS), D132.1 (VSS), D133.1 (VSS), D134.1 (VSS), D135.1 (VSS), D136.1 (VSS), D137.1 (VSS), D138.1 (VSS), D139.1 (VSS), D140.1 (VSS), D141.1 (VSS), D142.1 (VSS), D143.1 (VSS), D144.1 (VSS), D145.1 (VSS), D146.1 (VSS), D147.1 (VSS), D148.1 (VSS), D149.1 (VSS), D150.1 (VSS), D151.1 (VSS), D152.1 (VSS), D153.1 (VSS), D154.1 (VSS), D155.1 (VSS), D156.1 (VSS), D157.1 (VSS), D158.1 (VSS), D159.1 (VSS), D160.1 (VSS), D161.1 (VSS), D162.1 (VSS), D163.1 (VSS), D164.1 (VSS), D165.1 (VSS), D166.1 (VSS), D167.1 (VSS), D168.1 (VSS), D169.1 (VSS), D170.1 (VSS), D171.1 (VSS), D172.1 (VSS), D173.1 (VSS), D174.1 (VSS), D175.1 (VSS), D176.1 (VSS), D177.1 (VSS), D178.1 (VSS), D179.1 (VSS), D180.1 (VSS), D181.1 (VSS), D182.1 (VSS), D183.1 (VSS), D184.1 (VSS), D185.1 (VSS), D186.1 (VSS), D187.1 (VSS), D188.1 (VSS), D189.1 (VSS), D190.1 (VSS), D191.1 (VSS), D192.1 (VSS), D193.1 (VSS), D194.1 (VSS), D195.1 (VSS), D196.1 (VSS), D197.1 (VSS), D198.1 (VSS), D199.1 (VSS), D200.1 (VSS), D201.1 (VSS), D202.1 (VSS), D203.1 (VSS), D204.1 (VSS), D205.1 (VSS), D206.1 (VSS), D207.1 (VSS), D208.1 (VSS), D209.1 (VSS), D210.1 (VSS), D211.1 (VSS), D212.1 (VSS), D213.1 (VSS), D214.1 (VSS), D215.1 (VSS), D216.1 (VSS)
- net +5V: now reaches A1.40 (VBUS)
- net +5V: now also U1.9 (VDD), D109.3 (VDD), D110.3 (VDD), D111.3 (VDD), D112.3 (VDD), D113.3 (VDD), D114.3 (VDD), D115.3 (VDD), D116.3 (VDD), D117.3 (VDD), D118.3 (VDD), D119.3 (VDD), D120.3 (VDD), D121.3 (VDD), D122.3 (VDD), D123.3 (VDD), D124.3 (VDD), D125.3 (VDD), D126.3 (VDD), D127.3 (VDD), D128.3 (VDD), D129.3 (VDD), D130.3 (VDD), D131.3 (VDD), D132.3 (VDD), D133.3 (VDD), D134.3 (VDD), D135.3 (VDD), D136.3 (VDD), D137.3 (VDD), D138.3 (VDD), D139.3 (VDD), D140.3 (VDD), D141.3 (VDD), D142.3 (VDD), D143.3 (VDD), D144.3 (VDD), D145.3 (VDD), D146.3 (VDD), D147.3 (VDD), D148.3 (VDD), D149.3 (VDD), D150.3 (VDD), D151.3 (VDD), D152.3 (VDD), D153.3 (VDD), D154.3 (VDD), D155.3 (VDD), D156.3 (VDD), D157.3 (VDD), D158.3 (VDD), D159.3 (VDD), D160.3 (VDD), D161.3 (VDD), D162.3 (VDD), D163.3 (VDD), D164.3 (VDD), D165.3 (VDD), D166.3 (VDD), D167.3 (VDD), D168.3 (VDD), D169.3 (VDD), D170.3 (VDD), D171.3 (VDD), D172.3 (VDD), D173.3 (VDD), D174.3 (VDD), D175.3 (VDD), D176.3 (VDD), D177.3 (VDD), D178.3 (VDD), D179.3 (VDD), D180.3 (VDD), D181.3 (VDD), D182.3 (VDD), D183.3 (VDD), D184.3 (VDD), D185.3 (VDD), D186.3 (VDD), D187.3 (VDD), D188.3 (VDD), D189.3 (VDD), D190.3 (VDD), D191.3 (VDD), D192.3 (VDD), D193.3 (VDD), D194.3 (VDD), D195.3 (VDD), D196.3 (VDD), D197.3 (VDD), D198.3 (VDD), D199.3 (VDD), D200.3 (VDD), D201.3 (VDD), D202.3 (VDD), D203.3 (VDD), D204.3 (VDD), D205.3 (VDD), D206.3 (VDD), D207.3 (VDD), D208.3 (VDD), D209.3 (VDD), D210.3 (VDD), D211.3 (VDD), D212.3 (VDD), D213.3 (VDD), D214.3 (VDD), D215.3 (VDD), D216.3 (VDD)
- net OLED SCL: now reaches U1.21 (GPA0)
- net OLED SCL: now also J1.3 (Pin_3)
- net OLED SDA: now reaches U1.22 (GPA1)
- net OLED SDA: now also J1.4 (Pin_4)
- net LED DATA: now reaches U1.23 (GPA2)
- net LED DATA: now also D109.2 (DIN)
- net +3.3V: now reaches J1.2 (Pin_2)
- net +3.3V: now also A1.36 (3V3)
- net 3V3(OUT): no longer names the net of U1.18 (~{RESET})
- net 3V3(OUT): no longer A1.36 (3V3)
- new net: D110.4 (DOUT), D111.2 (DIN)
- new net: D111.4 (DOUT), D112.2 (DIN)
- new net: D165.2 (DIN), D168.4 (DOUT)
- new net: D163.2 (DIN), D165.4 (DOUT)
- new net: D144.4 (DOUT), D146.2 (DIN)
- new net: D146.4 (DOUT), D147.2 (DIN)
- new net: D128.4 (DOUT), D148.2 (DIN)
- new net: D145.2 (DIN), D148.4 (DOUT)
- new net: D121.4 (DOUT), D122.2 (DIN)
- new net: D122.4 (DOUT), D123.2 (DIN)
- new net: D120.4 (DOUT), D121.2 (DIN)
- new net: D158.4 (DOUT), D160.2 (DIN)
- new net: D160.4 (DOUT), D162.2 (DIN)
- new net: D109.4 (DOUT), D110.2 (DIN)
- new net: D179.2 (DIN), D181.4 (DOUT)
- new net: D177.2 (DIN), D179.4 (DOUT)
- new net: D201.2 (DIN), D203.4 (DOUT)
- new net: D199.2 (DIN), D201.4 (DOUT)
- new net: D214.2 (DIN), D215.4 (DOUT)
- new net: D213.2 (DIN), D214.4 (DOUT)
- new net: D184.4 (DOUT), D186.2 (DIN)
- new net: D186.4 (DOUT), D187.2 (DIN)
- new net: D197.2 (DIN), D199.4 (DOUT)
- new net: D195.2 (DIN), D197.4 (DOUT)
- new net: D151.2 (DIN), D153.4 (DOUT)
- new net: D150.2 (DIN), D151.4 (DOUT)
- new net: D130.2 (DIN), D131.4 (DOUT)
- new net: D129.2 (DIN), D130.4 (DOUT)
- new net: D124.4 (DOUT), D125.2 (DIN)
- new net: D125.4 (DOUT), D126.2 (DIN)
- new net: D187.4 (DOUT), D208.2 (DIN)
- new net: D205.2 (DIN), D208.4 (DOUT)
- new net: D164.4 (DOUT), D166.2 (DIN)
- new net: D166.4 (DOUT), D167.2 (DIN)
- new net: D149.4 (DOUT), D152.2 (DIN)
- new net: D152.4 (DOUT), D154.2 (DIN)
- new net: D167.4 (DOUT), D188.2 (DIN)
- new net: D142.4 (DOUT), D144.2 (DIN)
- new net: D211.2 (DIN), D212.4 (DOUT)
- new net: D210.2 (DIN), D211.4 (DOUT)
- new net: D174.4 (DOUT), D176.2 (DIN)
- new net: D176.4 (DOUT), D178.2 (DIN)
- new net: D147.4 (DOUT), D168.2 (DIN)
- new net: D149.2 (DIN), D150.4 (DOUT)
- new net: D191.2 (DIN), D193.4 (DOUT)
- new net: D190.2 (DIN), D191.4 (DOUT)
- new net: D126.4 (DOUT), D127.2 (DIN)
- new net: D112.4 (DOUT), D113.2 (DIN)
- new net: D113.4 (DOUT), D114.2 (DIN)
- new net: D132.4 (DOUT), D134.2 (DIN)
- new net: D134.4 (DOUT), D136.2 (DIN)
- new net: D139.2 (DIN), D141.4 (DOUT)
- new net: D137.2 (DIN), D139.4 (DOUT)
- new net: D189.4 (DOUT), D192.2 (DIN)
- new net: D192.4 (DOUT), D194.2 (DIN)
- new net: D193.2 (DIN), D195.4 (DOUT)
- new net: D123.4 (DOUT), D124.2 (DIN)
- new net: D203.2 (DIN), D205.4 (DOUT)
- new net: D140.4 (DOUT), D142.2 (DIN)
- new net: D129.4 (DOUT), D132.2 (DIN)
- new net: D159.2 (DIN), D161.4 (DOUT)
- new net: D157.2 (DIN), D159.4 (DOUT)
- new net: D194.4 (DOUT), D196.2 (DIN)
- new net: D212.2 (DIN), D213.4 (DOUT)
- new net: D135.2 (DIN), D137.4 (DOUT)
- new net: D156.4 (DOUT), D158.2 (DIN)
- new net: D185.2 (DIN), D188.4 (DOUT)
- new net: D183.2 (DIN), D185.4 (DOUT)
- new net: D162.4 (DOUT), D164.2 (DIN)
- new net: D202.4 (DOUT), D204.2 (DIN)
- new net: D204.4 (DOUT), D206.2 (DIN)
- new net: D133.2 (DIN), D135.4 (DOUT)
- new net: D131.2 (DIN), D133.4 (DOUT)
- new net: D189.2 (DIN), D190.4 (DOUT)
- new net: D178.4 (DOUT), D180.2 (DIN)
- new net: D180.4 (DOUT), D182.2 (DIN)
- new net: D196.4 (DOUT), D198.2 (DIN)
- new net: D114.4 (DOUT), D115.2 (DIN)
- new net: D115.4 (DOUT), D116.2 (DIN)
- new net: D127.4 (DOUT), D128.2 (DIN)
- new net: D119.4 (DOUT), D120.2 (DIN)
- new net: D182.4 (DOUT), D184.2 (DIN)
- new net: D161.2 (DIN), D163.4 (DOUT)
- new net: D143.2 (DIN), D145.4 (DOUT)
- new net: D141.2 (DIN), D143.4 (DOUT)
- new net: D169.2 (DIN), D170.4 (DOUT)
- new net: D169.4 (DOUT), D172.2 (DIN)
- new net: D215.2 (DIN), D216.4 (DOUT)
- new net: D181.2 (DIN), D183.4 (DOUT)
- new net: D206.4 (DOUT), D207.2 (DIN)
- new net: D209.2 (DIN), D210.4 (DOUT)
- new net: D172.4 (DOUT), D174.2 (DIN)
- new net: D173.2 (DIN), D175.4 (DOUT)
- new net: D171.2 (DIN), D173.4 (DOUT)
- new net: D170.2 (DIN), D171.4 (DOUT)
- new net: D154.4 (DOUT), D156.2 (DIN)
- new net: D116.4 (DOUT), D117.2 (DIN)
- new net: D207.4 (DOUT), D216.2 (DIN)
- new net: D175.2 (DIN), D177.4 (DOUT)
- new net: D155.2 (DIN), D157.4 (DOUT)
- new net: D153.2 (DIN), D155.4 (DOUT)
- new net: D117.4 (DOUT), D118.2 (DIN)
- new net: D136.4 (DOUT), D138.2 (DIN)
- new net: D138.4 (DOUT), D140.2 (DIN)
- new net: D118.4 (DOUT), D119.2 (DIN)
- new net: D198.4 (DOUT), D200.2 (DIN)
- new net: D200.4 (DOUT), D202.2 (DIN)

Commit message: resetting the submodules
Parts:
- added R1, R2, R3: 4.7k, easyeda2kicad:RES-TH_BD2.5-L4.7-P8.70-D0.5, symbol easyeda2kicad:RN16T24701F
- added SW109, SW110: RotaryEncoder_Switch, symbol Device:RotaryEncoder_Switch
- D1, D10, D100, D101, D102, D103, D104, D105, D106, D107, D108, D11, D12, D13, D14, D15, D16, D17, D18, D19, D2, D20, D21, D22, D23, D24, D25, D26, D27, D28, D29, D3, D30, D31, D32, D33, D34, D35, D36, D37, D38, D39, D4, D40, D41, D42, D43, D44, D45, D46, D47, D48, D49, D5, D50, D51, D52, D53, D54, D55, D56, D57, D58, D59, D6, D60, D61, D62, D63, D64, D65, D66, D67, D68, D69, D7, D70, D71, D72, D73, D74, D75, D76, D77, D78, D79, D8, D80, D81, D82, D83, D84, D85, D86, D87, D88, D89, D9, D90, D91, D92, D93, D94, D95, D96, D97, D98, D99: footprint (none) -> Diode_THT:D_DO-35_SOD27_P7.62mm_Horizontal
Connections:
- net +3.3V: now also R1.2, R2.2
- net +5V: now also R3.2
- net GND: now also SW109.C, SW110.C
- net LED DATA: now also U1.21 (GPA0); no longer U1.23 (GPA2)
- net SCL: now also J1.3 (Pin_3), R1.1
- net SDA: now also J1.4 (Pin_4), R2.1
- net RotEncoder1A: now reaches U1.1 (GPB0)
- net RotEncoder1A: now also SW109.A
- net at U1.18 (~{RESET}): now also R3.1
- net RotEncoder1B: now reaches U1.2 (GPB1)
- net RotEncoder1B: now also SW109.B
- net RotEncoder2B1: now reaches U1.24 (GPA3)
- net RotEncoder2B1: now also SW110.S1
- net RotEncoder2B2: now reaches U1.25 (GPA4)
- net RotEncoder2B2: now also SW110.S2
- net RotEncoder2A: now reaches U1.3 (GPB2)
- net RotEncoder2A: now also SW110.A
- net RotEncoder2B: now reaches U1.4 (GPB3)
- net RotEncoder2B: now also SW110.B
- removed net OLED SCL: J1.3 (Pin_3), U1.21 (GPA0)
- net OLED SDA renamed RotEncoder1B1
- net RotEncoder1B1: now also SW109.S1; no longer J1.4 (Pin_4)
- new net RotEncoder1B2: SW109.S2, U1.23 (GPA2)

Commit message: trying to add BOM and readded the keyswitch submodule
Parts:
- SW109, SW110: footprint (none) -> Rotary_Encoder:RotaryEncoder_Alps_EC11E-Switch_Vertical_H20mm
- SW95: footprint key-switches:SW_MX_Kailh_Choc_V1V2_THT_Hybrid -> Rotary_Encoder:RotaryEncoder_Alps_EC11E-Switch_Vertical_H20mm
Changed lines of the file:
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@@
 			)
 		)
-		(property "Footprint" ""
+		(property "Footprint" "Rotary_Encoder:RotaryEncoder_Alps_EC11E-Switch_Vertical_H20mm"
 			(at 304.8 172.466 0)
 			(effects
@@
 			)
 		)
-		(property "Footprint" "key-switches:SW_MX_Kailh_Choc_V1V2_THT_Hybrid"
+		(property "Footprint" "Rotary_Encoder:RotaryEncoder_Alps_EC11E-Switch_Vertical_H20mm"
 			(at 114.3 119.38 0)
 			(effects
@@
 			)
 		)
-		(property "Footprint" ""
+		(property "Footprint" "Rotary_Encoder:RotaryEncoder_Alps_EC11E-Switch_Vertical_H20mm"
 			(at 304.8 161.036 0)
 			(effects

Commit message: worked on laying out the keyboard
Parts:
- R1, R2, R3: footprint easyeda2kicad:RES-TH_BD2.5-L4.7-P8.70-D0.5 -> Resistor_THT:R_Axial_DIN0207_L6.3mm_D2.5mm_P2.54mm_Vertical
- SW109, SW110: footprint Rotary_Encoder:RotaryEncoder_Alps_EC11E-Switch_Vertical_H20mm -> easyeda2kicad:SW-TH_EC11XXXXXXXX
- U1: footprint Package_SO:SOIC-28W_7.5x17.9mm_P1.27mm -> Package_DIP:DIP-28_W7.62mm
Changed lines of the file:
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@@
 			)
 		)
-		(property "Footprint" "Rotary_Encoder:RotaryEncoder_Alps_EC11E-Switch_Vertical_H20mm"
+		(property "Footprint" "easyeda2kicad:SW-TH_EC11XXXXXXXX"
 			(at 304.8 172.466 0)
 			(effects
@@
 			)
 		)
-		(property "Footprint" "Package_SO:SOIC-28W_7.5x17.9mm_P1.27mm"
+		(property "Footprint" "Package_DIP:DIP-28_W7.62mm"
 			(at 373.38 149.86 0)
 			(effects
@@
 			)
 		)
-		(property "Footprint" "Rotary_Encoder:RotaryEncoder_Alps_EC11E-Switch_Vertical_H20mm"
+		(property "Footprint" "easyeda2kicad:SW-TH_EC11XXXXXXXX"
 			(at 304.8 161.036 0)
 			(effects
@@
 			)
 		)
-		(property "Footprint" "easyeda2kicad:RES-TH_BD2.5-L4.7-P8.70-D0.5"
+		(property "Footprint" "Resistor_THT:R_Axial_DIN0207_L6.3mm_D2.5mm_P2.54mm_Vertical"
 			(at 365.76 124.46 0)
 			(effects
@@
 			)
 		)
-		(property "Footprint" "easyeda2kicad:RES-TH_BD2.5-L4.7-P8.70-D0.5"
+		(property "Footprint" "Resistor_THT:R_Axial_DIN0207_L6.3mm_D2.5mm_P2.54mm_Vertical"
 			(at 356.87 129.54 0)
 			(effects
@@
 			)
 		)
-		(property "Footprint" "easyeda2kicad:RES-TH_BD2.5-L4.7-P8.70-D0.5"
+		(property "Footprint" "Resistor_THT:R_Axial_DIN0207_L6.3mm_D2.5mm_P2.54mm_Vertical"
 			(at 359.41 132.08 0)
 			(effects

Commit message: started laying out the pcb
Connections:
- net COL0: now also SW21.1; no longer SW19.1
- net COL1: now also SW22.1; no longer SW20.1
- net COL10: now also SW31.1; no longer SW29.1
- net COL11: now also SW32.1; no longer SW30.1
- net COL12: now also SW33.1; no longer SW31.1
- net COL13: now also SW34.1; no longer SW32.1
- net COL14: now also SW35.1; no longer SW33.1
- net COL15: now also SW36.1; no longer SW34.1
- net COL16: no longer SW35.1
- net COL17: no longer SW36.1
- net COL2: now also SW23.1; no longer SW21.1
- net COL3: now also SW24.1; no longer SW22.1
- net COL4: now also SW25.1; no longer SW23.1
- net COL5: now also SW26.1; no longer SW24.1
- net COL6: now also SW27.1; no longer SW25.1
- net COL7: now also SW28.1; no longer SW26.1
- net COL8: now also SW29.1; no longer SW27.1
- net COL9: now also SW30.1; no longer SW28.1
- net ROW1: no longer D19.1 (K), D20.1 (K)
Other:
- moved on the sheet: A1, D19, D20, D21, D22, D23, D24, D25, D26, D27, D28, D29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

Commit message: moved some keys on the matrix
re adjusting the keys on the matrix so they match there position on the keyboard.
Connections:
- net COL0: no longer SW1.1, SW21.1, SW37.1, SW55.1, SW73.1, SW91.1
- net COL1: no longer SW2.1, SW22.1, SW38.1, SW56.1, SW74.1, SW92.1
- net COL10: no longer SW101.1, SW11.1, SW31.1, SW47.1, SW65.1, SW83.1
- net COL11: no longer SW102.1, SW12.1, SW32.1, SW48.1, SW66.1, SW84.1
- net COL12: no longer SW103.1, SW13.1, SW33.1, SW49.1, SW67.1, SW85.1
- net COL13: no longer SW104.1, SW14.1, SW34.1, SW50.1, SW68.1, SW86.1
- net COL14: no longer SW105.1, SW15.1, SW35.1, SW51.1, SW69.1, SW87.1
- net COL15: no longer SW106.1, SW16.1, SW36.1, SW52.1, SW70.1, SW88.1
- net COL16: no longer SW107.1, SW17.1, SW53.1, SW71.1, SW89.1
- net COL17: no longer SW108.1, SW18.1, SW54.1, SW72.1, SW90.1
- net COL2: no longer SW23.1, SW3.1, SW39.1, SW57.1, SW75.1, SW93.1
- net COL3: no longer SW24.1, SW4.1, SW40.1, SW58.1, SW76.1, SW94.1
- net COL4: no longer SW25.1, SW41.1, SW5.1, SW59.1, SW77.1, SW95.1
- net COL5: no longer SW26.1, SW42.1, SW6.1, SW60.1, SW78.1, SW96.1
- net COL6: no longer SW27.1, SW43.1, SW61.1, SW7.1, SW79.1, SW97.1
- net COL7: no longer SW28.1, SW44.1, SW62.1, SW8.1, SW80.1, SW98.1
- net COL8: no longer SW29.1, SW45.1, SW63.1, SW81.1, SW9.1, SW99.1
- net COL9: no longer SW10.1, SW100.1, SW30.1, SW46.1, SW64.1, SW82.1
- net ROW0: no longer D1.1 (K), D10.1 (K), D11.1 (K), D12.1 (K), D13.1 (K), D14.1 (K), D15.1 (K), D16.1 (K), D17.1 (K), D18.1 (K), D2.1 (K), D3.1 (K), D4.1 (K), D5.1 (K), D6.1 (K), D7.1 (K), D8.1 (K), D9.1 (K)
- net ROW1: no longer D21.1 (K), D22.1 (K), D23.1 (K), D24.1 (K), D25.1 (K), D26.1 (K), D27.1 (K), D28.1 (K), D29.1 (K), D30.1 (K), D31.1 (K), D32.1 (K), D33.1 (K), D34.1 (K), D35.1 (K), D36.1 (K)
- net ROW2: no longer D37.1 (K), D38.1 (K), D39.1 (K), D40.1 (K), D41.1 (K), D42.1 (K), D43.1 (K), D44.1 (K), D45.1 (K), D46.1 (K), D47.1 (K), D48.1 (K), D49.1 (K), D50.1 (K), D51.1 (K), D52.1 (K), D53.1 (K), D54.1 (K)
- net ROW3: no longer D55.1 (K), D56.1 (K), D57.1 (K), D58.1 (K), D59.1 (K), D60.1 (K), D61.1 (K), D62.1 (K), D63.1 (K), D64.1 (K), D65.1 (K), D66.1 (K), D67.1 (K), D68.1 (K), D69.1 (K), D70.1 (K), D71.1 (K), D72.1 (K)
- net ROW4: no longer D73.1 (K), D74.1 (K), D75.1 (K), D76.1 (K), D77.1 (K), D78.1 (K), D79.1 (K), D80.1 (K), D81.1 (K), D82.1 (K), D83.1 (K), D84.1 (K), D85.1 (K), D86.1 (K), D87.1 (K), D88.1 (K), D89.1 (K), D90.1 (K)
- net ROW5: no longer D100.1 (K), D101.1 (K), D102.1 (K), D103.1 (K), D104.1 (K), D105.1 (K), D106.1 (K), D107.1 (K), D108.1 (K), D91.1 (K), D92.1 (K), D93.1 (K), D94.1 (K), D95.1 (K), D96.1 (K), D97.1 (K), D98.1 (K), D99.1 (K)
Other:
- moved on the sheet: D37, D38, D39, D40, D41, D42, D43, D44, D45, D46, D47, D48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
