File: PCB/full-keyboard.kicad_sch (KiCad schematic)
At the start: 332 parts, among them J1 Conn_01x04_Pin, SW1 SW_Push, SW10 SW_Push, SW100 SW_Push, SW101 SW_Push, SW102 SW_Push, SW103 SW_Push, SW104 SW_Push, SW105 SW_Push, SW106 SW_Push, SW107 SW_Push, SW108 SW_Push, SW109 RotaryEncoder_Switch, SW11 SW_Push, SW110 RotaryEncoder_Switch, SW12 SW_Push, SW13 SW_Push, SW14 SW_Push, SW15 SW_Push, SW16 SW_Push, SW17 SW_Push, SW18 SW_Push, SW19 SW_Push, SW2 SW_Push, SW20 SW_Push, SW21 SW_Push, SW22 SW_Push, SW23 SW_Push, SW24 SW_Push, SW25 SW_Push, SW26 SW_Push, SW27 SW_Push, SW28 SW_Push, SW29 SW_Push, SW3 SW_Push, SW30 SW_Push, SW31 SW_Push, SW32 SW_Push, SW33 SW_Push, SW34 SW_Push, SW35 SW_Push, SW36 SW_Push, SW37 SW_Push, SW38 SW_Push, SW39 SW_Push, SW4 SW_Push, SW40 SW_Push, SW41 SW_Push, SW42 SW_Push, SW43 SW_Push, SW44 SW_Push, SW45 SW_Push, SW46 SW_Push, SW47 SW_Push, SW48 SW_Push, SW49 SW_Push, SW5 SW_Push, SW50 SW_Push, SW51 SW_Push, SW52 SW_Push, SW53 SW_Push, SW54 SW_Push, SW55 SW_Push, SW56 SW_Push, SW57 SW_Push, SW58 SW_Push, SW59 SW_Push, SW6 SW_Push, SW60 SW_Push, SW61 SW_Push, SW62 SW_Push, SW63 SW_Push, SW64 SW_Push, SW65 SW_Push, SW66 SW_Push, SW67 SW_Push, SW68 SW_Push, SW69 SW_Push, SW7 SW_Push, SW70 SW_Push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

Commit message: set the layout in the schematic to match the pcb layout for the keys
Parts:
- removed SW110: RotaryEncoder_Switch, easyeda2kicad:SW-TH_EC11XXXXXXXX, symbol Device:RotaryEncoder_Switch
- SW95: footprint Rotary_Encoder:RotaryEncoder_Alps_EC11E-Switch_Vertical_H20mm -> key-switches:SW_MX_Kailh_Choc_V1V2_THT_Hybrid
Connections:
- net COL0: now also SW1.1, SW21.1, SW42.1, SW63.1, SW79.1, SW96.1
- net COL1: now also SW22.1, SW43.1, SW64.1, SW80.1, SW97.1
- net COL10: now also SW10.1, SW101.1, SW31.1, SW52.1, SW73.1, SW89.1
- net COL11: now also SW102.1, SW11.1, SW32.1, SW53.1, SW74.1, SW90.1
- net COL12: now also SW103.1, SW12.1, SW33.1, SW54.1, SW75.1
- net COL13: now also SW13.1, SW34.1, SW55.1
- net COL14: now also SW104.1, SW14.1, SW35.1, SW56.1
- net COL15: now also SW105.1, SW36.1, SW57.1, SW91.1
- net COL16: now also SW106.1, SW16.1, SW37.1, SW58.1
- net COL17: now also SW107.1, SW17.1, SW38.1, SW59.1, SW76.1, SW92.1
- net COL18: now also SW18.1, SW39.1, SW60.1, SW77.1, SW93.1
- net COL19: now also SW108.1, SW19.1, SW40.1, SW61.1, SW78.1, SW94.1
- net COL2: now also SW2.1, SW23.1, SW44.1, SW65.1, SW81.1, SW98.1
- net COL3: now also SW24.1, SW3.1, SW45.1, SW66.1, SW82.1
- net COL4: now also SW25.1, SW4.1, SW46.1, SW67.1, SW83.1
- net COL5: now also SW26.1, SW47.1, SW5.1, SW68.1, SW84.1
- net COL6: now also SW27.1, SW48.1, SW6.1, SW69.1, SW85.1, SW99.1
- net COL7: now also SW28.1, SW49.1, SW7.1, SW70.1, SW86.1
- net COL8: now also SW29.1, SW50.1, SW71.1, SW8.1, SW87.1
- net COL9: now also SW100.1, SW30.1, SW51.1, SW72.1, SW88.1, SW9.1
- net ROW0: now also D1.1 (K), D10.1 (K), D11.1 (K), D12.1 (K), D13.1 (K), D14.1 (K), D15.1 (K), D16.1 (K), D17.1 (K), D18.1 (K), D19.1 (K), D2.1 (K), D20.1 (K), D3.1 (K), D4.1 (K), D5.1 (K), D6.1 (K), D7.1 (K), D8.1 (K), D9.1 (K)
- net ROW1: now also D21.1 (K), D22.1 (K), D23.1 (K), D24.1 (K), D25.1 (K), D26.1 (K), D27.1 (K), D28.1 (K), D29.1 (K), D30.1 (K), D31.1 (K), D32.1 (K), D33.1 (K), D34.1 (K), D35.1 (K), D36.1 (K), D37.1 (K), D38.1 (K), D39.1 (K), D40.1 (K), D41.1 (K)
- net ROW2: now also D42.1 (K), D43.1 (K), D44.1 (K), D45.1 (K), D46.1 (K), D47.1 (K), D48.1 (K), D49.1 (K), D50.1 (K), D51.1 (K), D52.1 (K), D53.1 (K), D54.1 (K), D55.1 (K), D56.1 (K), D57.1 (K), D58.1 (K), D59.1 (K), D60.1 (K), D61.1 (K), D62.1 (K)
- net ROW3: now also D63.1 (K), D64.1 (K), D65.1 (K), D66.1 (K), D67.1 (K), D68.1 (K), D69.1 (K), D70.1 (K), D71.1 (K), D72.1 (K), D73.1 (K), D74.1 (K), D75.1 (K), D76.1 (K), D77.1 (K), D78.1 (K)
- net ROW4: now also D79.1 (K), D80.1 (K), D81.1 (K), D82.1 (K), D83.1 (K), D84.1 (K), D85.1 (K), D86.1 (K), D87.1 (K), D88.1 (K), D89.1 (K), D90.1 (K), D91.1 (K), D92.1 (K), D93.1 (K), D94.1 (K), D95.1 (K)
- net ROW5: now also D100.1 (K), D101.1 (K), D102.1 (K), D103.1 (K), D96.1 (K), D97.1 (K), D98.1 (K), D99.1 (K)
- net COL20: now reaches SW62.1
- net COL20: now also SW20.1, SW41.1, SW95.1
- net RotEncoder2A: no longer names the net of U1.3 (GPB2)
- net RotEncoder2B: no longer names the net of U1.4 (GPB3)
Other:
- moved on the sheet: D10, D104, D105, D106, D107, D108, D11, D12, D13, D14, D15, D16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

Commit message: changed the key matrix and started swapping keyswith libraries
Parts:
- added SW110: RotaryEncoder_Switch, easyeda2kicad:SW-TH_EC11XXXXXXXX, symbol Device:RotaryEncoder_Switch
Connections:
- net COL0: now also SW20.1, SW39.1, SW58.1, SW77.1; no longer SW21.1, SW42.1, SW63.1, SW79.1, SW96.1
- net COL1: now also SW2.1, SW21.1, SW40.1, SW59.1, SW78.1, SW96.1; no longer SW22.1, SW43.1, SW64.1, SW80.1, SW97.1
- net COL10: now also SW11.1, SW30.1, SW49.1, SW68.1, SW87.1; no longer SW10.1, SW31.1, SW52.1, SW73.1, SW89.1
- net COL11: now also SW12.1, SW31.1, SW50.1, SW69.1, SW88.1; no longer SW11.1, SW32.1, SW53.1, SW74.1, SW90.1
- net COL12: now also SW13.1, SW32.1, SW51.1, SW70.1, SW89.1; no longer SW12.1, SW33.1, SW54.1, SW75.1
- net COL13: now also SW14.1, SW33.1, SW52.1, SW71.1, SW90.1; no longer SW13.1, SW34.1, SW55.1
- net COL14: now also SW15.1, SW34.1, SW53.1, SW72.1, SW91.1; no longer SW14.1, SW35.1, SW56.1
- net COL15: now also SW16.1, SW35.1, SW54.1, SW73.1, SW92.1; no longer SW36.1, SW57.1, SW91.1
- net COL16: now also SW17.1, SW36.1, SW55.1, SW74.1, SW93.1; no longer SW16.1, SW37.1, SW58.1
- net COL17: now also SW18.1, SW37.1, SW56.1, SW75.1, SW94.1; no longer SW17.1, SW38.1, SW59.1, SW76.1, SW92.1
- net COL18: now also A1.25 (GPIO19), SW108.1, SW19.1, SW38.1, SW57.1, SW76.1, SW95.1; no longer SW18.1, SW39.1, SW60.1, SW77.1, SW93.1
- net COL2: now also SW22.1, SW3.1, SW41.1, SW60.1, SW79.1, SW97.1; no longer SW2.1, SW23.1, SW44.1, SW65.1, SW81.1, SW98.1
- net COL3: now also SW23.1, SW4.1, SW42.1, SW61.1, SW80.1, SW98.1; no longer SW24.1, SW3.1, SW45.1, SW66.1, SW82.1
- net COL4: now also SW24.1, SW43.1, SW5.1, SW62.1, SW81.1; no longer SW25.1, SW4.1, SW46.1, SW67.1, SW83.1
- net COL5: now also SW25.1, SW44.1, SW6.1, SW63.1, SW82.1; no longer SW26.1, SW47.1, SW5.1, SW68.1, SW84.1
- net COL6: now also SW26.1, SW45.1, SW64.1, SW7.1, SW83.1; no longer SW27.1, SW48.1, SW6.1, SW69.1, SW85.1
- net COL7: now also SW27.1, SW46.1, SW65.1, SW8.1, SW84.1; no longer SW28.1, SW49.1, SW7.1, SW70.1, SW86.1
- net COL8: now also SW28.1, SW47.1, SW66.1, SW85.1, SW9.1; no longer SW29.1, SW50.1, SW71.1, SW8.1, SW87.1
- net COL9: now also SW10.1, SW29.1, SW48.1, SW67.1, SW86.1; no longer SW30.1, SW51.1, SW72.1, SW88.1, SW9.1
- net GND: now also SW110.C
- net ROW0: now also A1.26 (GPIO20); no longer A1.25 (GPIO19), D20.1 (K)
- net ROW1: now also A1.27 (GPIO21), D20.1 (K); no longer A1.26 (GPIO20), D39.1 (K), D40.1 (K), D41.1 (K)
- net ROW2: now also A1.29 (GPIO22), D39.1 (K), D40.1 (K), D41.1 (K); no longer A1.27 (GPIO21), D58.1 (K), D59.1 (K), D60.1 (K), D61.1 (K), D62.1 (K)
- net ROW3: now also A1.31 (GPIO26_ADC0), D58.1 (K), D59.1 (K), D60.1 (K), D61.1 (K), D62.1 (K); no longer A1.29 (GPIO22), D77.1 (K), D78.1 (K)
- net ROW4: now also A1.32 (GPIO27_ADC1), D77.1 (K), D78.1 (K); no longer A1.31 (GPIO26_ADC0)
- net ROW5: now also A1.34 (GPIO28_ADC2), D104.1 (K), D105.1 (K), D106.1 (K), D107.1 (K), D108.1 (K); no longer A1.32 (GPIO27_ADC1)
- net RotEncoder2B1: now also U1.3 (GPB2), SW110.S1; no longer U1.24 (GPA3)
- net RotEncoder2B2: now also U1.4 (GPB3), SW110.S2; no longer U1.25 (GPA4)
- removed net COL19: SW108.1, SW19.1, SW40.1, SW61.1, SW78.1, SW94.1
- removed net COL20: SW20.1, SW41.1, SW62.1, SW95.1
- new net RotEncoder2A: SW110.A, U1.24 (GPA3)
- new net RotEncoder2B: SW110.B, U1.25 (GPA4)
Other:
- moved on the sheet: D10, D106, D108, D11, D12, D13, D14, D15, D16, D17, D18, D19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

Commit message: got the leds placed into position
Parts:
- D109, D110, D111, D112, D113, D114, D115, D116, D117, D118, D119, D120, D121, D122, D123, D124, D125, D126, D127, D128, D129, D130, D131, D132, D133, D134, D135, D136, D137, D138, D139, D140, D141, D142, D143, D144, D145, D146, D147, D148, D149, D150, D151, D152, D153, D154, D155, D156, D157, D158, D159, D160, D161, D162, D163, D164, D165, D166, D167, D168, D169, D170, D171, D172, D173, D174, D175, D176, D177, D178, D179, D180, D181, D182, D183, D184, D185, D186, D187, D188, D189, D190, D191, D192, D193, D194, D195, D196, D197, D198, D199, D200, D201, D202, D203, D204, D205, D206, D207, D208, D209, D210, D211, D212, D213, D214, D215, D216: footprint LED_SMD:LED_SK6812_PLCC4_5.0x5.0mm_P3.2mm -> custom1:MX_SK6812MINI-E_REV
- J1: footprint KiCad-SSD1306-0.91-OLED-4pin-128x32:SSD1306-0.91-OLED-4pin-128x32 -> custom1:SSD1306-0.91-OLED-4pin-128x32
- SW1, SW10, SW104, SW105, SW106, SW108, SW11, SW12, SW13, SW14, SW15, SW16, SW17, SW18, SW19, SW2, SW20, SW21, SW22, SW23, SW24, SW25, SW26, SW27, SW28, SW29, SW3, SW30, SW31, SW32, SW33, SW35, SW36, SW37, SW38, SW39, SW4, SW40, SW41, SW43, SW44, SW45, SW46, SW47, SW48, SW49, SW5, SW50, SW51, SW52, SW53, SW54, SW56, SW57, SW58, SW59, SW6, SW60, SW61, SW64, SW65, SW66, SW67, SW68, SW69, SW7, SW70, SW71, SW72, SW73, SW74, SW76, SW77, SW78, SW8, SW80, SW81, SW82, SW83, SW84, SW85, SW86, SW87, SW88, SW89, SW9, SW91, SW92, SW93, SW94: footprint key-switches:SW_MX_Kailh_Choc_V1V2_THT_Hybrid -> PCM_Switch_Keyboard_Hotswap_Kailh:SW_Hotswap_Kailh_MX_1.00u
- SW100, SW101, SW102, SW103, SW96, SW97, SW98: footprint key-switches:SW_MX_Kailh_Choc_V1V2_THT_Hybrid -> PCM_Switch_Keyboard_Hotswap_Kailh:SW_Hotswap_Kailh_MX_1.25u
- SW107, SW34: footprint key-switches:SW_MX_Kailh_Choc_V1V2_THT_Hybrid -> PCM_Switch_Keyboard_Hotswap_Kailh:SW_Hotswap_Kailh_MX_2.00u
- SW42, SW55: footprint key-switches:SW_MX_Kailh_Choc_V1V2_THT_Hybrid -> PCM_Switch_Keyboard_Hotswap_Kailh:SW_Hotswap_Kailh_MX_1.50u
- SW62, SW95: footprint key-switches:SW_MX_Kailh_Choc_V1V2_THT_Hybrid -> PCM_Switch_Keyboard_Hotswap_Kailh:SW_Hotswap_Kailh_MX_2.00u_90deg
- SW63: footprint key-switches:SW_MX_Kailh_Choc_V1V2_THT_Hybrid -> PCM_Switch_Keyboard_Hotswap_Kailh:SW_Hotswap_Kailh_MX_1.75u
- SW75, SW79: footprint key-switches:SW_MX_Kailh_Choc_V1V2_THT_Hybrid -> PCM_Switch_Keyboard_Hotswap_Kailh:SW_Hotswap_Kailh_MX_2.25u
- SW90: footprint key-switches:SW_MX_Kailh_Choc_V1V2_THT_Hybrid -> PCM_Switch_Keyboard_Hotswap_Kailh:SW_Hotswap_Kailh_MX_2.75u
- SW99: footprint key-switches:SW_MX_Kailh_Choc_V1V2_THT_Hybrid -> PCM_Switch_Keyboard_Hotswap_Kailh:SW_Hotswap_Kailh_MX_6.25u
