File: PCB/full-keyboard.kicad_pcb (KiCad board)
At the start: 2 copper layers, 3.4 x 3 mm, 332 parts, among them J1 Conn_01x04_Pin, SW1 SW_Push, SW10 SW_Push, SW100 SW_Push, SW101 SW_Push, SW102 SW_Push, SW103 SW_Push, SW104 SW_Push, SW105 SW_Push, SW106 SW_Push, SW107 SW_Push, SW108 SW_Push, SW109 RotaryEncoder_Switch, SW11 SW_Push, SW110 RotaryEncoder_Switch, SW12 SW_Push, SW13 SW_Push, SW14 SW_Push, SW15 SW_Push, SW16 SW_Push, SW17 SW_Push, SW18 SW_Push, SW19 SW_Push, SW2 SW_Push, SW20 SW_Push, SW21 SW_Push, SW22 SW_Push, SW23 SW_Push, SW24 SW_Push, SW25 SW_Push, SW26 SW_Push, SW27 SW_Push, SW28 SW_Push, SW29 SW_Push, SW3 SW_Push, SW30 SW_Push, SW31 SW_Push, SW32 SW_Push, SW33 SW_Push, SW34 SW_Push, SW35 SW_Push, SW36 SW_Push, SW37 SW_Push, SW38 SW_Push, SW39 SW_Push, SW4 SW_Push, SW40 SW_Push, SW41 SW_Push, SW42 SW_Push, SW43 SW_Push, SW44 SW_Push, SW45 SW_Push, SW46 SW_Push, SW47 SW_Push, SW48 SW_Push, SW49 SW_Push, SW5 SW_Push, SW50 SW_Push, SW51 SW_Push, SW52 SW_Push, SW53 SW_Push, SW54 SW_Push, SW55 SW_Push, SW56 SW_Push, SW57 SW_Push, SW58 SW_Push, SW59 SW_Push, SW6 SW_Push, SW60 SW_Push, SW61 SW_Push, SW62 SW_Push, SW63 SW_Push, SW64 SW_Push, SW65 SW_Push, SW66 SW_Push, SW67 SW_Push, SW68 SW_Push, SW69 SW_Push, SW7 SW_Push, SW70 SW_Push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

Commit message: macking sure changes where backed up.
Parts:
- added REF**: SW_Hotswap_Kailh_MX_1.00u, PCM_Switch_Keyboard_Hotswap_Kailh:SW_Hotswap_Kailh_MX_1.00u, F.Cu at (267.1, 39.6)
- D109: moved to F.Cu
- SW107: footprint CherryMX_KailhSocket_StabWireTop_LTST-A683CEGBW-Rotated-HS:CherryMX_2.00u_KailhSocket_StabWireTop_LTST-A683CEGBW-Rotate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 -> PCM_Switch_Keyboard_Hotswap_Kailh:SW_Hotswap_Kailh_MX_2.00u
- SW34: footprint PCM_Switch_Keyboard_Hotswap_Kailh:SW_Hotswap_Kailh_MX_1.00u -> PCM_Switch_Keyboard_Hotswap_Kailh:SW_Hotswap_Kailh_MX_2.00u
- SW55: footprint PCM_Switch_Keyboard_Hotswap_Kailh:SW_Hotswap_Kailh_MX_1.00u -> PCM_Switch_Keyboard_Hotswap_Kailh:SW_Hotswap_Kailh_MX_1.50u
- SW75: footprint PCM_Switch_Keyboard_Hotswap_Kailh:SW_Hotswap_Kailh_MX_1.00u -> PCM_Switch_Keyboard_Hotswap_Kailh:SW_Hotswap_Kailh_MX_2.25u
- SW90: footprint PCM_Switch_Keyboard_Hotswap_Kailh:SW_Hotswap_Kailh_MX_1.00u -> PCM_Switch_Keyboard_Hotswap_Kailh:SW_Hotswap_Kailh_MX_2.75u
- SW99: footprint PCM_Switch_Keyboard_Hotswap_Kailh:SW_Hotswap_Kailh_MX_1.00u -> PCM_Switch_Keyboard_Hotswap_Kailh:SW_Hotswap_Kailh_MX_6.25u
- moved D110 228.2 mm to (86.0, 70.0), turned to 0 degrees
- moved D121 72.6 mm to (176.8, 286.9), turned to 0 degrees
- moved D213 72.6 mm to (241.8, 207.5), turned to 0 degrees
- moved D122 65.9 mm to (184.9, 207.5), turned to 0 degrees
- moved D134 65.9 mm to (184.9, 286.9), turned to 0 degrees
- moved D212 65.9 mm to (233.6, 286.9), turned to 0 degrees
- moved D200 65.9 mm to (233.6, 207.5), turned to 0 degrees
- moved D120 65.6 mm to (176.8, 280.3), turned to 0 degrees
- moved D214 65.6 mm to (241.8, 214.1), turned to 0 degrees
- moved D199 60.7 mm to (225.5, 286.9), turned to 0 degrees
- moved D147 60.7 mm to (193.0, 286.9), turned to 0 degrees
- moved D135 60.7 mm to (193.0, 207.5), turned to 0 degrees
- moved D187 60.7 mm to (225.5, 207.5), turned to 0 degrees
- moved D111 59.3 mm to (176.8, 220.7), turned to 0 degrees
- moved D119 59.3 mm to (176.8, 273.7), turned to 0 degrees
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Other:
- board outline removed
