File: PCB/full-keyboard.kicad_pcb (KiCad board)
At the start: 2 copper layers, 333 parts, among them J1 Conn_01x04_Pin, SW1 SW_Push, SW10 SW_Push, SW100 SW_Push, SW101 SW_Push, SW102 SW_Push, SW103 SW_Push, SW104 SW_Push, SW105 SW_Push, SW106 SW_Push, SW107 SW_Push, SW108 SW_Push, SW109 RotaryEncoder_Switch, SW11 SW_Push, SW110 RotaryEncoder_Switch, SW12 SW_Push, SW13 SW_Push, SW14 SW_Push, SW15 SW_Push, SW16 SW_Push, SW17 SW_Push, SW18 SW_Push, SW19 SW_Push, SW2 SW_Push, SW20 SW_Push, SW21 SW_Push, SW22 SW_Push, SW23 SW_Push, SW24 SW_Push, SW25 SW_Push, SW26 SW_Push, SW27 SW_Push, SW28 SW_Push, SW29 SW_Push, SW3 SW_Push, SW30 SW_Push, SW31 SW_Push, SW32 SW_Push, SW33 SW_Push, SW34 SW_Push, SW35 SW_Push, SW36 SW_Push, SW37 SW_Push, SW38 SW_Push, SW39 SW_Push, SW4 SW_Push, SW40 SW_Push, SW41 SW_Push, SW42 SW_Push, SW43 SW_Push, SW44 SW_Push, SW45 SW_Push, SW46 SW_Push, SW47 SW_Push, SW48 SW_Push, SW49 SW_Push, SW5 SW_Push, SW50 SW_Push, SW51 SW_Push, SW52 SW_Push, SW53 SW_Push, SW54 SW_Push, SW55 SW_Push, SW56 SW_Push, SW57 SW_Push, SW58 SW_Push, SW59 SW_Push, SW6 SW_Push, SW60 SW_Push, SW61 SW_Push, SW62 SW_Push, SW63 SW_Push, SW64 SW_Push, SW65 SW_Push, SW66 SW_Push, SW67 SW_Push, SW68 SW_Push, SW69 SW_Push, SW7 SW_Push, SW70 SW_Push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

Commit message: finnished placing the keyswitches properly and started working on placing the leds
Parts:
- removed REF**: SW_Hotswap_Kailh_MX_1.00u, PCM_Switch_Keyboard_Hotswap_Kailh:SW_Hotswap_Kailh_MX_1.00u
- SW100, SW101, SW102, SW103, SW96, SW97, SW98: footprint CherryMX_PCB_KailhSocket_LED:CherryMX_1.25u_PCB_KailhSocket_LED -> PCM_Switch_Keyboard_Hotswap_Kailh:SW_Hotswap_Kailh_MX_1.25u
- SW42: footprint CherryMX_PCB_KailhSocket_LED:CherryMX_1.50u_PCB_KailhSocket_LED -> PCM_Switch_Keyboard_Hotswap_Kailh:SW_Hotswap_Kailh_MX_1.50u
- SW62: footprint PCM_Switch_Keyboard_Hotswap_Kailh:SW_Hotswap_Kailh_MX_1.00u -> PCM_Switch_Keyboard_Hotswap_Kailh:SW_Hotswap_Kailh_MX_2.00u_90deg
- SW63: footprint CherryMX_PCB_KailhSocket_LED:CherryMX_1.75u_PCB_KailhSocket_LED -> PCM_Switch_Keyboard_Hotswap_Kailh:SW_Hotswap_Kailh_MX_1.75u
- SW79: footprint CherryMX_PCB_KailhSocket_LED:CherryMX_2.25u_PCB_KailhSocket_LED -> PCM_Switch_Keyboard_Hotswap_Kailh:SW_Hotswap_Kailh_MX_2.25u
- moved D128 323.9 mm to (456.1, 70.0)
- moved D129 312.6 mm to (456.3, 98.6)
- moved D127 304.5 mm to (437.1, 69.9)
- moved D130 299.6 mm to (437.1, 98.7)
- moved D131 287.7 mm to (418.1, 98.5)
- moved D126 285.4 mm to (418.3, 69.7)
- moved D170 283.7 mm to (456.2, 127.4)
- moved D132 276.7 mm to (399.1, 98.5)
- moved A1 270.7 mm to (442.7, 41.4), turned to -90 degrees
- moved D169 269.0 mm to (437.4, 117.8)
- moved D171 265.9 mm to (437.2, 136.8)
- moved D125 265.0 mm to (398.8, 70.8)
- moved D133 263.1 mm to (375.2, 98.6)
- moved D121 256.2 mm to (313.6, 70.3)
- moved D134 254.6 mm to (356.3, 98.6)
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
Commit message: got the leds placed into position
Parts:
- D109, D110, D111, D112, D113, D114, D115, D116, D117, D118, D119, D120, D121, D122, D123, D124, D125, D126, D127, D128, D129, D130, D131, D132, D133, D134, D135, D136, D137, D138, D139, D140, D141, D142, D143, D144, D145, D146, D147, D148, D149, D150, D151, D152, D153, D154, D155, D156, D157, D158, D159, D160, D161, D162, D163, D164, D165, D166, D167, D168, D169, D170, D171, D172, D173, D174, D175, D176, D177, D178, D179, D180, D181, D182, D183, D184, D185, D186, D187, D188, D189, D190, D191, D192, D193, D194, D195, D196, D197, D198, D199, D200, D201, D202, D203, D204, D205, D206, D207, D208, D209, D210, D211, D212, D213, D214, D215, D216: footprint LED_SMD:LED_SK6812_PLCC4_5.0x5.0mm_P3.2mm -> custom1:MX_SK6812MINI-E_REV
- J1: footprint KiCad-SSD1306-0.91-OLED-4pin-128x32:SSD1306-0.91-OLED-4pin-128x32 -> custom1:SSD1306-0.91-OLED-4pin-128x32
- moved D1 346.8 mm to (57.3, 67.0)
- moved D2 321.2 mm to (94.2, 67.1)
- moved D3 310.1 mm to (113.0, 67.0)
- moved D4 298.9 mm to (132.4, 67.0)
- moved D5 288.2 mm to (151.5, 67.2)
- moved D6 272.4 mm to (179.9, 67.1)
- moved D7 263.1 mm to (199.2, 67.0)
- moved D186 257.1 mm to (53.4, 131.2)
- moved D8 254.3 mm to (218.2, 67.2)
- moved D9 246.4 mm to (237.3, 67.2)
- moved D14 244.8 mm to (315.3, 44.9)
- moved D15 244.8 mm to (318.9, 44.9)
- moved D16 244.8 mm to (322.4, 44.9)
- moved D17 244.8 mm to (325.9, 44.9)
- moved D18 244.8 mm to (329.5, 44.9)
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Connections:
- U1 pad 24: unconnected-(U1-GPA3-Pad24) -> /RotEncoder2A
- U1 pad 25: unconnected-(U1-GPA4-Pad25) -> /RotEncoder2B
- U1 pad 3: unconnected-(U1-GPB2-Pad3) -> /RotEncoder2B1
- U1 pad 4: unconnected-(U1-GPB3-Pad4) -> /RotEncoder2B2
Other:
- board outline added: 3.6 x 3.3 mm
