File: PCB/full-keyboard.kicad_pcb (KiCad board)
At the start: 2 copper layers, 434 x 161.7 mm, 232 parts, among them J1 Conn_01x04_Pin, SW1 SW_Push, SW10 SW_Push, SW100 SW_Push, SW101 SW_Push, SW102 SW_Push, SW103 SW_Push, SW104 SW_Push, SW105 SW_Push, SW106 SW_Push, SW107 SW_Push, SW108 SW_Push, SW109 RotaryEncoder_Switch, SW11 SW_Push, SW110 RotaryEncoder_Switch, SW12 SW_Push, SW13 SW_Push, SW14 SW_Push, SW15 SW_Push, SW16 SW_Push, SW17 SW_Push, SW18 SW_Push, SW19 SW_Push, SW2 SW_Push, SW20 SW_Push, SW21 SW_Push, SW22 SW_Push, SW23 SW_Push, SW24 SW_Push, SW25 SW_Push, SW26 SW_Push, SW27 SW_Push, SW28 SW_Push, SW29 SW_Push, SW3 SW_Push, SW30 SW_Push, SW31 SW_Push, SW32 SW_Push, SW33 SW_Push, SW34 SW_Push, SW35 SW_Push, SW36 SW_Push, SW37 SW_Push, SW38 SW_Push, SW39 SW_Push, SW4 SW_Push, SW40 SW_Push, SW41 SW_Push, SW42 SW_Push, SW43 SW_Push, SW44 SW_Push, SW45 SW_Push, SW46 SW_Push, SW47 SW_Push, SW48 SW_Push, SW49 SW_Push, SW5 SW_Push, SW50 SW_Push, SW51 SW_Push, SW52 SW_Push, SW53 SW_Push, SW54 SW_Push, SW55 SW_Push, SW56 SW_Push, SW57 SW_Push, SW58 SW_Push, SW59 SW_Push, SW6 SW_Push, SW60 SW_Push, SW61 SW_Push, SW62 SW_Push, SW63 SW_Push, SW64 SW_Push, SW65 SW_Push, SW66 SW_Push, SW67 SW_Push, SW68 SW_Push, SW69 SW_Push, SW7 SW_Push, SW70 SW_Push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

Commit message: added case model
Parts:
- R3: footprint easyeda2kicad:RES-TH_BD2.5-L4.7-P8.70-D0.5 -> Resistor_THT:R_Axial_DIN0204_L3.6mm_D1.6mm_P1.90mm_Vertical
- SW100, SW101, SW102, SW103, SW96, SW97, SW98: footprint PCM_Switch_Keyboard_Cherry_MX:SW_Cherry_MX_Plate_1.25u -> PCM_Switch_Keyboard_Cherry_MX:SW_Cherry_MX_PCB_1.25u
- SW107, SW34: footprint PCM_Switch_Keyboard_Cherry_MX:SW_Cherry_MX_Plate_2.00u -> PCM_Switch_Keyboard_Cherry_MX:SW_Cherry_MX_PCB_2.00u
- SW42, SW55: footprint PCM_Switch_Keyboard_Cherry_MX:SW_Cherry_MX_Plate_1.50u -> PCM_Switch_Keyboard_Cherry_MX:SW_Cherry_MX_PCB_1.50u
- SW62, SW95: footprint PCM_Switch_Keyboard_Cherry_MX:SW_Cherry_MX_Plate_2.00u_90deg -> PCM_Switch_Keyboard_Cherry_MX:SW_Cherry_MX_PCB_2.00u_90deg
- SW63: footprint PCM_Switch_Keyboard_Cherry_MX:SW_Cherry_MX_Plate_1.75u -> PCM_Switch_Keyboard_Cherry_MX:SW_Cherry_MX_PCB_1.75u
- SW75, SW79: footprint PCM_Switch_Keyboard_Cherry_MX:SW_Cherry_MX_Plate_2.25u -> PCM_Switch_Keyboard_Cherry_MX:SW_Cherry_MX_PCB_2.25u
- SW90: footprint PCM_Switch_Keyboard_Cherry_MX:SW_Cherry_MX_Plate_2.75u -> PCM_Switch_Keyboard_Cherry_MX:SW_Cherry_MX_PCB_2.75u
- SW99: footprint PCM_Switch_Keyboard_Cherry_MX:SW_Cherry_MX_Plate_6.25u -> PCM_Switch_Keyboard_Cherry_MX:SW_Cherry_MX_PCB_6.25u
- moved R3 3.73 mm to (401.7, 36.8)
Routing:
- net /COL3: track 182.8 -> 966.5 mm, vias 0 -> 9
- net /COL1: track 291.9 -> 1033.5 mm, vias 4 -> 13
- net /COL0: track 318.6 -> 1053.4 mm, vias 7 -> 16
- net /COL4: track 179.6 -> 882.9 mm, vias 0 -> 9
- net /COL2: track 301.0 -> 1003.6 mm, vias 4 -> 13
- net /COL5: track 240.2 -> 929.8 mm, vias 0 -> 7
- net /COL6: track 238.8 -> 892.1 mm, vias 0 -> 9
- net /COL7: track 202.2 -> 850.4 mm, vias 0 -> 9
- net /COL9: track 163.2 -> 739.6 mm, vias 0 -> 12
- net /COL8: track 313.8 -> 741.1 mm, vias 0 -> 5
- net /ROW6: track 140.5 -> 496.1 mm, vias 0 -> 5
- net /ROW4: track 158.0 -> 495.6 mm, vias 0 -> 6
- net /ROW9: track 294.7 -> 576.8 mm, vias 0 -> 6
- net /ROW2: track 171.5 -> 435.0 mm, vias 0 -> 4
- net /ROW7: track 259.0 -> 493.6 mm, vias 0 -> 4
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Other:
- board size 434 x 161.7 mm -> 434 x 166.8 mm

Commit message: switched to case made by TurboCase for a nicer case with standoff.
Parts:
- added ?: , TurboCase:Cutout_TypeC, F.Cu at (471.0, 43.4)
- added REF**: MountingHole_2.2mm_M2, MountingHole:MountingHole_2.2mm_M2, F.Cu at (241.0, 184.6)
- added REF**: MountingHole_2.2mm_M2, MountingHole:MountingHole_2.2mm_M2, F.Cu at (39.0, 184.4)
- added REF**: MountingHole_2.2mm_M2, MountingHole:MountingHole_2.2mm_M2, F.Cu at (466.0, 23.8)
- added REF**: MountingHole_2.2mm_M2, MountingHole:MountingHole_2.2mm_M2, F.Cu at (38.4, 23.8)
- added REF**: MountingHole_2.2mm_M2, MountingHole:MountingHole_2.2mm_M2, F.Cu at (466.0, 184.6)
- added REF**: MountingHole_2.2mm_M2, MountingHole:MountingHole_2.2mm_M2, F.Cu at (238.6, 29.0)
Routing:
- net /COL8: track 741.1 -> 740.3 mm

Commit message: made the case in FreeCAD and moved the locations of two of the mounting holes and added a 7th
Parts:
- added REF**: MountingHole_2.2mm_M2, MountingHole:MountingHole_2.2mm_M2, F.Cu at (326.0, 131.6)
- moved REF** 13.7 mm to (252.2, 30.6)
- moved REF** 11.2 mm to (252.2, 184.6)
Routing:
- net /COL6: track 892.1 -> 887.4 mm
- net /COL1: track 1033.5 -> 1029.1 mm
- net /COL7: track 850.4 -> 846.2 mm
- net /ROW7: track 493.6 -> 489.7 mm
- net /COL8: track 740.3 -> 736.7 mm
- net /COL0: track 1053.4 -> 1049.9 mm
- net /COL5: track 929.8 -> 926.4 mm
- net /COL4: track 882.9 -> 880.1 mm
- net /COL2: track 1003.6 -> 1000.9 mm
- net /COL3: track 966.5 -> 963.9 mm
- net GND: track 229.9 -> 227.9 mm
- net /ROW6: track 496.1 -> 494.4 mm
- net /ROW4: track 495.6 -> 494.1 mm
- net /COL9: track 739.6 -> 738.1 mm
- net +3.3V: track 210.3 -> 209.1 mm
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